File: a2b_d/a2b.kicad_pcb (KiCad board)
At the start: 2 copper layers, 58.4 x 66.7 mm, 16 parts, among them SW1 SW_DIP_x03, SW2 SW_DIP_x03, SW3 SW_DIP_x02

Commit message: Move Library Files to a central location: 2026-07-14 14:52:11
Parts:
- DC_IN1: footprint RAPC722X:SWITCHCRAFT_RAPC722X -> Library:SWITCHCRAFT_RAPC722X
Changed lines of the file:
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@@
 		)
 	)
-	(footprint "RAPC722X:SWITCHCRAFT_RAPC722X"
+	(footprint "Library:SWITCHCRAFT_RAPC722X"
 		(layer "F.Cu")
 		(at 147.59 76.935 180)
 		(property "Reference" "DC_IN1"
-			(at -1.02125 -8.89 0)
+			(at -0.97875 -8.89 0)
 			(layer "F.SilkS")
 			(effects
@@
 		(fp_line
 			(start 3.5 7.49)
+			(end 3.5 -0.905)
+			(stroke
+				(width 0.127)
+				(type solid)
+			)
+			(layer "F.SilkS")
+		)
+		(fp_line
+			(start 3.5 -5.595)
+			(end 3.5 -7.01)
+			(stroke
+				(width 0.127)
+				(type solid)
+			)
+			(layer "F.SilkS")
+		)
+		(fp_line
+			(start 3.5 -7.01)
+			(end 1.6 -7.01)
+			(stroke
+				(width 0.127)
+				(type solid)
+			)
+			(layer "F.SilkS")
+		)
+		(fp_line
+			(start -3.6 -7.01)
+			(end -5.5 -7.01)
+			(stroke
+				(width 0.127)
+				(type solid)
+			)
+			(layer "F.SilkS")
+		)
+		(fp_line
+			(start -5.5 7.49)
+			(end 3.5 7.49)
+			(stroke
+				(width 0.127)
+				(type solid)
+			)
+			(layer "F.SilkS")
+		)
+		(fp_line
+			(start -5.5 -7.01)
 			(end -5.5 7.49)
 			(stroke
@@
 		)
 		(fp_line
+			(start 5.0625 -0.975)
+			(end 5.0625 -5.525)
+			(stroke
+				(width 0.05)
+				(type solid)
+			)
+			(layer "F.CrtYd")
+		)
+		(fp_line
+			(start 5.0625 -5.525)
+			(end 3.75 -5.525)
+			(stroke
+				(width 0.05)
+				(type solid)
+			)
+			(layer "F.CrtYd")
+		)
+		(fp_line
+			(start 3.75 7.74)
+			(end 3.75 -0.975)
+			(stroke
+				(width 0.05)
+				(type solid)
+			)
+			(layer "F.CrtYd")
+		)
+		(fp_line
+			(start 3.75 -0.975)
+			(end 5.0625 -0.975)
+			(stroke
+				(width 0.05)
+				(type solid)
+			)
+			(layer "F.CrtYd")
+		)
+		(fp_line
+			(start 3.75 -5.525)
+			(end 3.75 -7.64)
+			(stroke
+				(width 0.05)
+				(type solid)
+			)
+			(layer "F.CrtYd")
+		)
+		(fp_line
+			(start 3.75 -7.64)
+			(end -5.75 -7.64)
+			(stroke
+				(width 0.05)
+				(type solid)
+			)
+			(layer "F.CrtYd")
+		)
+		(fp_line
+			(start -5.75 7.74)
+			(end 3.75 7.74)
+			(stroke
+				(width 0.05)
+				(type solid)
+			)
+			(layer "F.CrtYd")
+		)
+		(fp_line
+			(start -5.75 -0.95)
+			(end -5.75 7.74)
+			(stroke
+				(width 0.05)
+				(type solid)
+			)
+			(layer "F.CrtYd")
+		)
+		(fp_line
+			(start -5.75 -7.64)
+			(end -5.75 -5.5)
+			(stroke
+				(width 0.05)
+				(type solid)
+			)
+			(layer "F.CrtYd")
+		)
+		(fp_line
+			(start -7.0625 -0.95)
+			(end -5.75 -0.95)
+			(stroke
+				(width 0.05)
+				(type solid)
+			)
+			(layer "F.CrtYd")
+		)
+		(fp_line
+			(start -7.0625 -5.5)
+			(end -5.75 -5.5)
+			(stroke
+				(width 0.05)
+				(type solid)
+			)
+			(layer "F.CrtYd")
+		)
+		(fp_line
+			(start -7.0625 -5.5)
+			(end -7.0625 -0.95)
+			(stroke
+				(width 0.05)
+				(type solid)
+			)
+			(layer "F.CrtYd")
+		)
+		(fp_line
+			(start 3.5 7.49)
+			(end 3.5 -7.01)
+			(stroke
+				(width 0.127)
+				(type solid)
+			)
+			(layer "F.Fab")
+		)
+		(fp_line
 			(start 3.5 -7.01)
+			(end -5.5 -7.01)
+			(stroke
+				(width 0.127)
+				(type solid)
+			)
+			(layer "F.Fab")
+		)
+		(fp_line
+			(start -5.5 7.49)
 			(end 3.5 7.49)
 			(stroke
@@
 				(type solid)
 			)
-			(layer "F.SilkS")
-		)
-		(fp_line
-			(start 1.6 -7.01)
-			(end 3.5 -7.01)
-			(stroke
-				(width 0.127)
-				(type solid)
-			)
-			(layer "F.SilkS")
-		)
-		(fp_line
-			(start -5.5 7.49)
-			(end -5.5 -0.905)
-			(stroke
-				(width 0.127)
-				(type solid)
-			)
-			(layer "F.SilkS")
-		)
-		(fp_line
-			(start -5.5 -5.595)
-			(end -5.5 -7.01)
-			(stroke
-				(width 0.127)
-				(type solid)
-			)
-			(layer "F.SilkS")
+			(layer "F.Fab")
 		)
 		(fp_line
 			(start -5.5 -7.01)
-			(end -3.6 -7.01)
-			(stroke
-				(width 0.127)
-				(type solid)
-			)
-			(layer "F.SilkS")
-		)
-		(fp_line
-			(start 3.75 7.74)
-			(end -5.75 7.74)
-			(stroke
-				(width 0.05)
-				(type solid)
-			)
-			(layer "F.CrtYd")
-		)
-		(fp_line
-			(start 3.75 -7.64)
-			(end 3.75 7.74)
-			(stroke
-				(width 0.05)
-				(type solid)
-			)
-			(layer "F.CrtYd")
-		)
-		(fp_line
-			(start -5.75 7.74)
-			(end -5.75 -0.975)
-			(stroke
-				(width 0.05)
-				(type solid)
-			)
-			(layer "F.CrtYd")
-		)
-		(fp_line
-			(start -5.75 -0.975)
-			(end -7.0625 -0.975)
-			(stroke
-				(width 0.05)
-				(type solid)
-			)
-			(layer "F.CrtYd")
-		)
-		(fp_line
-			(start -5.75 -5.525)
-			(end -5.75 -7.64)
-			(stroke
-				(width 0.05)
-				(type solid)
-			)
-			(layer "F.CrtYd")
-		)
-		(fp_line
-			(start -5.75 -7.64)
-			(end 3.75 -7.64)
-			(stroke
-				(width 0.05)
-				(type solid)
-			)
-			(layer "F.CrtYd")
-		)
-		(fp_line
-			(start -7.0625 -0.975)
-			(end -7.0625 -5.525)
-			(stroke
-				(width 0.05)
-				(type solid)
-			)
-			(layer "F.CrtYd")
-		)
-		(fp_line
-			(start -7.0625 -5.525)
-			(end -5.75 -5.525)
-			(stroke
-				(width 0.05)
-				(type solid)
-			)
-			(layer "F.CrtYd")
-		)
-		(fp_line
-			(start 3.5 7.49)
 			(end -5.5 7.49)
-			(stroke
-				(width 0.127)
-				(type solid)
-			)
-			(layer "F.Fab")
-		)
-		(fp_line
-			(start 3.5 -7.01)
-			(end 3.5 7.49)
-			(stroke
-				(width 0.127)
-				(type solid)
-			)
-			(layer "F.Fab")
-		)
-		(fp_line
-			(start -5.5 7.49)
-			(end -5.5 -7.01)
-			(stroke
-				(width 0.127)
-				(type solid)
-			)
-			(layer "F.Fab")
-		)
-		(fp_line
-			(start -5.5 -7.01)
-			(end 3.5 -7.01)
 			(stroke
 				(width 0.127)
@@
 			(solder_mask_margin 0.102)
 		)
+		(pad "SHUNT" thru_hole oval
+			(at 3.8 -3.25 180)
+			(size 2.025 4.05)
+			(drill oval 0.76 3.05)
+			(layers "*.Cu" "*.Mask")
+			(remove_unused_layers no)
+			(solder_mask_margin 0.102)
+		)
 		(pad "SLEEVE" thru_hole oval
 			(at -1 0 180)
@@
 		)
 		(embedded_fonts no)
-		(model "${KIPRJMOD}/My_Library/3d Models/RAPC722X.step"
+		(model "${KIPRJMOD}/../My_Library/3d Models/RAPC722X.step"
 			(offset
-				(xyz -1 -7.5 -1.5)
+				(xyz -1 -7.4 -1.5)
 			)
 			(scale
@@
 			)
 			(rotate
-				(xyz 90 -0 180)
-			)
-		)
+				(xyz 90 -180 180)
+			)
+		)
