File: a2b_u/a2b.kicad_pcb (KiCad board)
At the start: 2 copper layers, 58.4 x 66.7 mm, 16 parts, among them SW1 SW_DIP_x03, SW2 SW_DIP_x03, SW3 SW_DIP_x02

Commit message: Move Library Files to a central location: 2026-07-14 14:52:11
Changed lines of the file:
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@@
 	(footprint "RAPC722X:SWITCHCRAFT_RAPC722X"
 		(layer "F.Cu")
-		(at 147.59 76.935 180)
+		(at 147.5851 76.935 180)
 		(property "Reference" "DC_IN1"
 			(at -0.97875 -8.89 0)
@@
 		(sheetname "/")
 		(sheetfile "a2b.kicad_sch")
-		(units
-			(unit
-				(name "A")
-				(pins "PIN" "SHUNT" "SLEEVE")
-			)
-		)
 		(attr through_hole)
 		(duplicate_pad_numbers_are_jumpers no)
@@
 		)
 		(fp_line
-			(start -5.75 -7.64)
+			(start -5.75 -0.95)
 			(end -5.75 7.74)
 			(stroke
@@
 		)
 		(fp_line
+			(start -5.75 -7.64)
+			(end -5.75 -5.5)
+			(stroke
+				(width 0.05)
+				(type solid)
+			)
+			(layer "F.CrtYd")
+		)
+		(fp_line
+			(start -7.0625 -0.95)
+			(end -5.75 -0.95)
+			(stroke
+				(width 0.05)
+				(type solid)
+			)
+			(layer "F.CrtYd")
+		)
+		(fp_line
+			(start -7.0625 -5.5)
+			(end -5.75 -5.5)
+			(stroke
+				(width 0.05)
+				(type solid)
+			)
+			(layer "F.CrtYd")
+		)
+		(fp_line
+			(start -7.0625 -5.5)
+			(end -7.0625 -0.95)
+			(stroke
+				(width 0.05)
+				(type solid)
+			)
+			(layer "F.CrtYd")
+		)
+		(fp_line
 			(start 3.5 7.49)
 			(end 3.5 -7.01)
@@
 		)
 		(pad "SHUNT" thru_hole oval
+			(at -5.8 -3.25 180)
+			(size 2.025 4.05)
+			(drill oval 0.76 3.05)
+			(layers "*.Cu" "*.Mask")
+			(remove_unused_layers no)
+			(pintype "passive")
+			(solder_mask_margin 0.102)
+		)
+		(pad "SHUNT" thru_hole oval
 			(at 3.8 -3.25 180)
 			(size 2.025 4.05)
@@
 		(model "${KIPRJMOD}/My_Library/3d Models/RAPC722X.step"
 			(offset
-				(xyz -1 -7.5 -0.5)
+				(xyz -1 -7.4 -1.5)
 			)
 			(scale
@@
 	)
 	(segment
-		(start 148.59 78.2492)
-		(end 145.141162 81.698038)
+		(start 145.415 81.4242)
+		(end 145.415 88.4332)
 		(width 0.2)
 		(layer "F.Cu")
@@
 	)
 	(segment
-		(start 145.141162 81.698038)
-		(end 145.141162 88.159362)
+		(start 147.3201 90.3383)
+		(end 147.3201 91.44)
 		(width 0.2)
 		(layer "F.Cu")
@@
 	)
 	(segment
-		(start 148.59 76.935)
-		(end 148.59 78.2492)
+		(start 148.59 78.2492)
+		(end 145.415 81.4242)
 		(width 0.2)
 		(layer "F.Cu")
@@
 	)
 	(segment
-		(start 147.3201 90.3383)
-		(end 147.3201 91.44)
+		(start 148.59 76.935)
+		(end 148.59 78.2492)
 		(width 0.2)
 		(layer "F.Cu")
@@
 	)
 	(segment
-		(start 145.141162 88.159362)
+		(start 145.415 88.4332)
 		(end 147.3201 90.3383)
 		(width 0.2)
