File: a2b_u/a2b.kicad_sch (KiCad schematic)
At the start: 16 parts, among them SW1 SW_DIP_x03, SW2 SW_DIP_x03, SW3 SW_DIP_x02

Commit message: Move Library Files to a central location: 2026-07-14 14:52:11
Parts:
- D1, D2: KiLib_Generator (none) -> LED/THT
- R1: KiLib_Generator (none) -> resistor/THT
Changed lines of the file:
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@@
+			)
+		)
+		(property "KiLib_Generator" "LED/THT"
+			(at 127 87.63 0)
+			(hide yes)
+			(show_name no)
+			(do_not_autoplace no)
+			(effects
+				(font
+					(size 1.27 1.27)
+				)
 			)
 		)
@@
 			)
 		)
+		(property "ok" ""
+			(at 127 44.45 0)
+			(hide yes)
+			(show_name no)
+			(do_not_autoplace no)
+			(effects
+				(font
+					(size 1.27 1.27)
+				)
+			)
+		)
 		(pin "SHUNT"
 		)
@@
 			)
 		)
+		(property "KiLib_Generator" "resistor/THT"
+			(at 133.35 100.33 0)
+			(hide yes)
+			(show_name no)
+			(do_not_autoplace no)
+			(effects
+				(font
+					(size 1.27 1.27)
+				)
+			)
+		)
 		(pin "1"
 		)
@@
 			(hide yes)
 			(show_name no)
+			(do_not_autoplace no)
+			(effects
+				(font
+					(size 1.27 1.27)
+				)
+			)
+		)
+		(property "KiLib_Generator" "LED/THT"
+			(at 133.35 87.63 0)
+			(hide yes)
+			(show_name no)
